File: PCB/Open-ESPilot/Open-ESPilot-Peripheral.kicad_sch (KiCad schematic)
At the start: 24 parts, among them J10 GND, J11 RC in, J12 LED out, J13 Micro_SD_Card, J14 Micro SD Card, J4 UART0, J5 UART1, J6 UART2, J7 I2C, J8 PWM output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

Commit message: Schematic Fixes
Parts:
- added JP10, JP11, JP12, JP13, JP14, JP15, JP16, JP17, JP18, JP19, JP20, JP21, JP22, JP23, JP24, JP25, JP26, JP27, JP28, JP6, JP7, JP8, JP9: R_Small, Jumper:SolderJumper-2_P1.3mm_Bridged2Bar_RoundedPad1.0x1.5mm, symbol Device:R_Small
Connections:
- net ADC-Voltage: now also JP12.1
- net BUZZER: now also JP18.1
- net GPIO14: now also JP15.2; no longer J13.5 (CLK), J14.5 (Pin_5)
- net GPIO15: now also JP14.2; no longer J13.3 (CMD), J14.3 (Pin_3)
- net GPIO16: now also JP6.2; no longer J6.5 (Pin_5)
- net GPIO17: now also JP7.2; no longer J6.6 (Pin_6)
- net GPIO18: now also JP17.2; no longer D1.4 (DIN)
- net GPIO2: now also JP16.2; no longer J13.7 (DAT0), J14.7 (Pin_7)
- net GPIO21: now also JP13.2; no longer JP2.2 (C)
- net GPIO35: now also JP21.2; no longer J8.1 (Pin_1)
- net GPIO36: now also JP22.2; no longer J8.2 (Pin_2)
- net GPIO37: now also JP23.2; no longer J8.3 (Pin_3)
- net GPIO38: now also JP24.2; no longer J8.4 (Pin_4)
- net GPIO39: now also JP25.2; no longer J8.5 (Pin_5)
- net GPIO40: now also JP26.2; no longer J8.6 (Pin_6)
- net GPIO41: now also JP27.2; no longer J8.7 (Pin_7)
- net GPIO42: now also JP28.2; no longer J8.8 (Pin_8)
- net GPIO43: now also JP11.2; no longer J4.1 (Pin_1)
- net GPIO44: now also JP10.2; no longer J4.2 (Pin_2)
- net GPIO6: now also JP9.2; no longer J5.1 (Pin_1)
- net GPIO7: now also JP8.2; no longer J5.2 (Pin_2)
- net SCL: now also JP19.1
- net SDA: now also JP20.1
- new net GPIO4: JP12.2
- new net GPIO47: JP19.2
- new net GPIO48: JP20.2
- new net GPIO8: JP18.2
- new net LED: D1.4 (DIN), JP17.1
- new net RCin: JP13.1, JP2.2 (C)
- new net SD-CLK: J13.5 (CLK), J14.5 (Pin_5), JP15.1
- new net SD-CMD: J13.3 (CMD), J14.3 (Pin_3), JP14.1
- new net SD-DAT0: J13.7 (DAT0), J14.7 (Pin_7), JP16.1
- new net ServoOutput1: J8.1 (Pin_1), JP21.1
- new net ServoOutput2: J8.2 (Pin_2), JP22.1
- new net ServoOutput3: J8.3 (Pin_3), JP23.1
- new net ServoOutput4: J8.4 (Pin_4), JP24.1
- new net ServoOutput5: J8.5 (Pin_5), JP25.1
- new net ServoOutput6: J8.6 (Pin_6), JP26.1
- new net ServoOutput7: J8.7 (Pin_7), JP27.1
- new net ServoOutput8: J8.8 (Pin_8), JP28.1
- new net U0-RX: J4.2 (Pin_2), JP10.1
- new net U0-TX: J4.1 (Pin_1), JP11.1
- new net U1-RX: J5.2 (Pin_2), JP8.1
- new net U1-TX: J5.1 (Pin_1), JP9.1
- new net U2-RX: J6.6 (Pin_6), JP7.1
- new net U2-TX: J6.5 (Pin_5), JP6.1
Other:
- moved on the sheet: J10, J13, J4, J5, J6, J7, J8, J9, JP1, JP2, R10, R11
