File: PCB/Open-ESPilot/Open-ESPilot-Peripheral.kicad_sch (KiCad schematic)
At the start: 58 parts, among them J10 UART1, J11 UART2, J12 I2C, J14 LED out, J5 PWM output, J6 RC in, J7 Vx, J8 GND, J9 UART0, M2 GY91, Q2 BC847, Q3 BC847, U5 Micro_SD_Card

Commit message: Selected componets and tried to made a csv.
Parts:
- C15, C17, C18, C19, C20, C21, C22, C23, C24: LCSC (none) -> C49678
- C16: LCSC (none) -> C5674
- D5: LCSC (none) -> C2843785
- J10, J11, J12, J14, J5, J6, J7, J8, J9, JP10, JP11, JP12, JP13, JP14, JP15, JP16, JP17, JP18, JP19, JP20, JP21, JP22, JP23, JP24, JP25, JP26, JP27, JP28, JP4, JP5, JP6, JP7, JP8, JP9, TP6, TP7, TP8: LCSC (none) -> -
- M2: LCSC (none) -> -; Non LCSC link (none) -> https://www.aliexpress.com/item/32652866365.html
- R13: LCSC (none) -> C84376
- R14, R15, R16, R17: LCSC (none) -> C95781

Commit message: in dabenginging of V1.1
Parts:
- U5: symbol Connector:Micro_SD_Card -> Connector:Micro_SD_Card_Det_Hirose_DM3AT
- renumbered JP27 to GJ14, JP26 to GJ15, JP20 to GJ16, JP21 to GJ17, JP24 to GJ18, JP28 to GJ2, JP12 to GJ21, JP4 to GJ35, JP5 to GJ36, JP6 to GJ37, JP7 to GJ38, JP8 to GJ39, JP15 to GJ4, JP9 to GJ40, JP10 to GJ41, JP11 to GJ42, JP16 to GJ43, JP17 to GJ44, JP23 to GJ47, JP22 to GJ48, JP18 to GJ6, JP19 to GJ7, JP25 to GJ8, JP14 to JP4, JP13 to JP5
Connections:
- net +3V3: now also R13.1
- net +5V: no longer JP4.2 (B), R13.1
- net GND: now also U5.11 (SHIELD); no longer U5.9 (SHIELD)
- new net +5Vreg: JP4.2 (B)
- no-connect marks 1 -> 3
Other:
- note added: "Power the PWM outpu with a battery"

Commit message: PCB init of V1.1
Other:
- note added: "Power the PWM output with a battery"
- note removed: "Power the PWM outpu with a battery"
- company: (none) -> Tomas Kuchta
Changed lines of the file:
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@@
 		(title "Open-ESPilot")
 		(rev "V1.1")
+		(company "Tomas Kuchta")
 	)
 	(rectangle
@@
 		)
 	)
-	(text "Power the PWM outpu with a battery"
+	(text "Power the PWM output with a battery"
 		(exclude_from_sim no)
 		(at 70.358 74.168 0)
