File: PCB/Open-ESPilot/Open-ESPilot-MCU.kicad_sch (KiCad schematic)
At the start: 18 parts, among them J1 USB_C_Receptacle_USB2.0_16P, SW1 SW_Push, SW2 SW_Push, U1 ESP32-S3-WROOM-1-N8

Commit message: I'm rushing it! :( Finished the PCB
Parts:
- TP5: footprint TestPoint:TestPoint_THTPad_D2.0mm_Drill1.0mm -> TestPoint:TestPoint_Pad_D2.0mm
Connections:
- net +3V3: now also R3.1
- net +3V3p: no longer R3.1
Changed lines of the file:
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@@
 		)
 	)
-	(label "+3V3p"
+	(label "+3V3"
 		(at 208.28 113.03 270)
 		(effects
@@
 			)
 		)
-		(property "Footprint" "TestPoint:TestPoint_THTPad_D2.0mm_Drill1.0mm"
+		(property "Footprint" "TestPoint:TestPoint_Pad_D2.0mm"
 			(at 73.66 58.42 0)
 			(effects

Commit message: Selected componets and tried to made a csv.
Parts:
- C1, C3: LCSC (none) -> C49678
- C4: LCSC (none) -> C5674
- R1, R2: LCSC (none) -> C84375
- R3, R4: LCSC (none) -> C84376
- TP1, TP2, TP3, TP4, TP5: LCSC (none) -> -
- U1: LCSC (none) -> C2913198
Changed lines of the file:
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@@
+			)
+		)
+		(property "LCSC" "C84375"
+			(at 200.66 76.2 0)
+			(effects
+				(font
+					(size 1.27 1.27)
+				)
+				(hide yes)
 			)
 		)
@@
 			)
 		)
+		(property "LCSC" "C5674"
+			(at 247.65 138.43 0)
+			(effects
+				(font
+					(size 1.27 1.27)
+				)
+				(hide yes)
+			)
+		)
 		(pin "2"
 		)
@@
 			)
 		)
+		(property "LCSC" "-"
+			(at 73.66 53.34 90)
+			(effects
+				(font
+					(size 1.27 1.27)
+				)
+				(hide yes)
+			)
+		)
 		(pin "1"
 		)
@@
 		(property "Description" "test point"
 			(at 73.66 39.37 0)
+			(effects
+				(font
+					(size 1.27 1.27)
+				)
+				(hide yes)
+			)
+		)
+		(property "LCSC" "-"
+			(at 73.66 39.37 90)
 			(effects
 				(font
@@
 			)
 		)
+		(property "LCSC" "-"
+			(at 73.66 35.56 90)
+			(effects
+				(font
+					(size 1.27 1.27)
+				)
+				(hide yes)
+			)
+		)
 		(pin "1"
 		)
@@
 		)
 		(property "Function" "Decoupling"
+			(at 148.59 36.83 0)
+			(effects
+				(font
+					(size 1.27 1.27)
+				)
+				(hide yes)
+			)
+		)
+		(property "LCSC" "C49678"
 			(at 148.59 36.83 0)
 			(effects
@@
 			)
 		)
+		(property "LCSC" "C84375"
+			(at 208.28 76.2 0)
+			(effects
+				(font
+					(size 1.27 1.27)
+				)
+				(hide yes)
+			)
+		)
 		(pin "1"
 		)
@@
 			)
 		)
+		(property "LCSC" "C84376"
+			(at 255.27 124.46 0)
+			(effects
+				(font
+					(size 1.27 1.27)
+				)
+				(hide yes)
+			)
+		)
 		(pin "1"
 		)
@@
 			)
 		)
+		(property "LCSC" "C49678"
+			(at 200.66 138.43 0)
+			(effects
+				(font
+					(size 1.27 1.27)
+				)
+				(hide yes)
+			)
+		)
 		(pin "2"
 		)
@@
 		(property "Description" "test point"
 			(at 73.66 43.18 0)
+			(effects
+				(font
+					(size 1.27 1.27)
+				)
+				(hide yes)
+			)
+		)
+		(property "LCSC" "-"
+			(at 73.66 43.18 90)
 			(effects
 				(font
@@
 			)
 		)
+		(property "LCSC" "C2913198"
+			(at 72.39 139.7 0)
+			(effects
+				(font
+					(size 1.27 1.27)
+				)
+				(hide yes)
+			)
+		)
 		(pin "8"
 		)
@@
 		(property "Description" "test point"
 			(at 73.66 49.53 0)
+			(effects
+				(font
+					(size 1.27 1.27)
+				)
+				(hide yes)
+			)
+		)
+		(property "LCSC" "-"
+			(at 73.66 49.53 90)
 			(effects
 				(font
@@
 			(at 208.28 124.46 0)
 			(effects
+				(font
+					(size 1.27 1.27)
+				)
+				(hide yes)
+			)
+		)
+		(property "LCSC" "C84376"
+			(at 208.28 124.46 0)
+			(effects

Commit message: in dabenginging of V1.1
Other:
- moved on the sheet: FB1
Changed lines of the file:
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@@
 	(title_block
 		(title "Open-ESPilot")
+		(rev "V1.1")
 	)
 	(rectangle
@@
 	)
 	(junction
+		(at 162.56 184.15)
+		(diameter 0)
+		(color 0 0 0 0)
+	)
+	(junction
 		(at 255.27 130.81)
 		(diameter 0)
@@
 		)
 	)
+	(wire
+		(pts
+			(xy 162.56 181.61) (xy 162.56 184.15)
+		)
+		(stroke
+			(width 0)
+			(type default)
+		)
+	)
 	(bus
 		(pts
@@
 	(wire
 		(pts
-			(xy 144.78 177.8) (xy 151.13 177.8)
+			(xy 144.78 184.15) (xy 151.13 184.15)
 		)
 		(stroke
@@
 	(wire
 		(pts
-			(xy 156.21 177.8) (xy 163.83 177.8)
+			(xy 156.21 184.15) (xy 162.56 184.15)
 		)
 		(stroke
@@
 	(wire
 		(pts
+			(xy 162.56 184.15) (xy 163.83 184.15)
+		)
+		(stroke
+			(width 0)
+			(type default)
+		)
+	)
+	(wire
+		(pts
 			(xy 208.28 72.39) (xy 208.28 62.23)
 		)
@@
 	)
 	(label "+3V3p"
-		(at 163.83 177.8 0)
+		(at 163.83 184.15 0)
 		(effects
 			(font
@@
 	(hierarchical_label "+3V3"
 		(shape input)
-		(at 144.78 177.8 180)
+		(at 144.78 184.15 180)
 		(effects
 			(font
@@
 		)
 		(instances
-			(project ""
+			(project "Open-ESPilot"
 				(path "/2992e60d-a645-4cd7-90ae-fe72311b6bee/83c0ee2d-1731-42ff-aa2e-45ac54ea980d"
 					(reference "#PWR012")
@@
 		)
 		(instances
-			(project ""
+			(project "Open-ESPilot"
 				(path "/2992e60d-a645-4cd7-90ae-fe72311b6bee/83c0ee2d-1731-42ff-aa2e-45ac54ea980d"
 					(reference "C4")
@@
 		)
 		(instances
-			(project ""
+			(project "Open-ESPilot"
 				(path "/2992e60d-a645-4cd7-90ae-fe72311b6bee/83c0ee2d-1731-42ff-aa2e-45ac54ea980d"
 					(reference "#PWR09")
@@
 		)
 		(instances
-			(project ""
+			(project "Open-ESPilot"
 				(path "/2992e60d-a645-4cd7-90ae-fe72311b6bee/83c0ee2d-1731-42ff-aa2e-45ac54ea980d"
 					(reference "TP1")
@@
 		)
 		(instances
-			(project ""
+			(project "Open-ESPilot"
 				(path "/2992e60d-a645-4cd7-90ae-fe72311b6bee/83c0ee2d-1731-42ff-aa2e-45ac54ea980d"
 					(reference "R2")
@@
 	)
 	(symbol
+		(lib_id "power:PWR_FLAG")
+		(at 162.56 181.61 0)
+		(unit 1)
+		(exclude_from_sim no)
+		(in_bom yes)
+		(on_board yes)
+		(dnp no)
+		(property "Reference" "#FLG06"
+			(at 162.56 179.705 0)
+			(effects
+				(font
+					(size 1.27 1.27)
+				)
+				(hide yes)
+			)
+		)
+		(property "Value" "PWR_FLAG"
+			(at 162.56 178.054 90)
+			(effects
+				(font
+					(size 1.27 1.27)
+				)
+				(justify left)
+			)
+		)
+		(property "Footprint" ""
+			(at 162.56 181.61 0)
+			(effects
+				(font
+					(size 1.27 1.27)
+				)
+				(hide yes)
+			)
+		)
+		(property "Datasheet" "~"
+			(at 162.56 181.61 0)
+			(effects
+				(font
+					(size 1.27 1.27)
+				)
+				(hide yes)
+			)
+		)
+		(property "Description" "Special symbol for telling ERC where power comes from"
+			(at 162.56 181.61 0)
+			(effects
+				(font
+					(size 1.27 1.27)
+				)
+				(hide yes)
+			)
+		)
+		(pin "1"
+		)
+		(instances
+			(project "Open-ESPilot"
+				(path "/2992e60d-a645-4cd7-90ae-fe72311b6bee/83c0ee2d-1731-42ff-aa2e-45ac54ea980d"
+					(reference "#FLG06")
+					(unit 1)
+				)
+			)
+		)
+	)
+	(symbol
 		(lib_id "Switch:SW_Push")
 		(at 208.28 138.43 90)
@@
 		)
 		(instances
-			(project ""
+			(project "Open-ESPilot"
 				(path "/2992e60d-a645-4cd7-90ae-fe72311b6bee/83c0ee2d-1731-42ff-aa2e-45ac54ea980d"
 					(reference "SW1")
@@
 		)
 		(instances
-			(project ""
+			(project "Open-ESPilot"
 				(path "/2992e60d-a645-4cd7-90ae-fe72311b6bee/83c0ee2d-1731-42ff-aa2e-45ac54ea980d"
 					(reference "#PWR010")
@@
 		)
 		(instances
-			(project ""
+			(project "Open-ESPilot"
 				(path "/2992e60d-a645-4cd7-90ae-fe72311b6bee/83c0ee2d-1731-42ff-aa2e-45ac54ea980d"
 					(reference "U1")
@@
 		)
 		(instances
-			(project ""
+			(project "Open-ESPilot"
 				(path "/2992e60d-a645-4cd7-90ae-fe72311b6bee/83c0ee2d-1731-42ff-aa2e-45ac54ea980d"
 					(reference "R3")
@@
 	(symbol
 		(lib_id "Device:FerriteBead_Small")
-		(at 153.67 177.8 90)
+		(at 153.67 184.15 90)
 		(unit 1)
 		(exclude_from_sim no)
@@
 		(fields_autoplaced yes)
 		(property "Reference" "FB1"
-			(at 153.6319 171.45 90)
+			(at 153.6319 177.8 90)
 			(effects
 				(font
@@
 		)
 		(property "Value" "FerriteBead"
-			(at 153.6319 173.99 90)
+			(at 153.6319 180.34 90)
 			(effects
 				(font
@@
 		)
 		(property "Footprint" "Inductor_SMD:L_0805_2012Metric_Pad1.05x1.20mm_HandSolder"
-			(at 153.67 179.578 90)
+			(at 153.67 185.928 90)
 			(effects
 				(font
@@
 		)
 		(property "Datasheet" "~"
-			(at 153.67 177.8 0)
+			(at 153.67 184.15 0)
 			(effects
 				(font
@@
 		)
 		(property "Description" "Ferrite bead, small symbol"
-			(at 153.67 177.8 0)
+			(at 153.67 184.15 0)
 			(effects
 				(font
@@
 		)
 		(property "LCSC" "C15957"
-			(at 153.67 177.8 90)
+			(at 153.67 184.15 90)
 			(effects
 				(font
@@
 		)
 		(instances
-			(project ""
+			(project "Open-ESPilot"
 				(path "/2992e60d-a645-4cd7-90ae-fe72311b6bee/83c0ee2d-1731-42ff-aa2e-45ac54ea980d"
 					(reference "FB1")
@@
 		)
 		(instances
-			(project ""
+			(project "Open-ESPilot"
 				(path "/2992e60d-a645-4cd7-90ae-fe72311b6bee/83c0ee2d-1731-42ff-aa2e-45ac54ea980d"
 					(reference "#PWR06")
@@
 		)
 		(instances
-			(project ""
+			(project "Open-ESPilot"
 				(path "/2992e60d-a645-4cd7-90ae-fe72311b6bee/83c0ee2d-1731-42ff-aa2e-45ac54ea980d"
 					(reference "J1")
