File: PCB/Open-ESPilot/Open-ESPilot.kicad_pcb (KiCad board)
At the start: 2 copper layers, 50.6 x 71.1 mm, 109 parts, among them J1 USB_C_Receptacle_USB2.0_16P, J10 UART1, J11 UART2, J12 I2C, J14 LED out, J2 VOUT, J3 VIN, J4 GND, J5 PWM output, J6 RC in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

Commit message: PCB init of V1.1
Parts:
- moved JP4 3.21 mm to (186.5, 85.5)
Other:
- board text added: "VERSION 1.1"
- board text removed: "VERSION 1"
Changed lines of the file:
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@@
 	)
 	(paper "A4")
+	(title_block
+		(title "Open-ESPilot")
+		(rev "V1.1")
+		(company "Tomas Kuchta")
+	)
 	(layers
 		(0 "F.Cu" signal)
@@
 	(footprint "Jumper:SolderJumper-2_P1.3mm_Bridged2Bar_RoundedPad1.0x1.5mm"
 		(layer "F.Cu")
-		(at 185.35 88.5)
+		(at 186.5 85.5)
 		(descr "SMD Solder Jumper, 1x1.5mm, rounded Pads, 0.3mm gap, bridged with 2 copper strips")
 		(tags "net tie solder jumper bridged")
@@
 		)
 	)
-	(gr_text "VERSION 1"
+	(gr_text "VERSION 1.1"
 		(at 166 127 0)
 		(layer "B.SilkS")
